Commit message: binder changes

File: resources/SM_Cup.urdf (robot description, URDF)
Before this commit: robot jeroen_cup_object, 1 links, 0 joints
Links:
- removed link jeroen_cup_main
- added link SM_Cup_main, mass 0.1; collision mesh filename=/home/user/catkin_init_ws/src/pycram/resources/SM_Cup.stl scale=1 1 1; visual mesh filename=/home/user/catkin_init_ws/src/pycram/resources/SM_Cup.stl scale=1 1 1

File: resources/bowl.urdf (robot description, URDF)
Before this commit: robot SM_Cup_object, 1 links, 0 joints
Links:
- removed link SM_Cup_main
- added link bowl_main, mass 0.1; collision mesh filename=/home/user/catkin_init_ws/src/pycram/resources/bowl.stl scale=1 1 1; visual mesh filename=/home/user/catkin_init_ws/src/pycram/resources/bowl.stl scale=1 1 1

File: resources/milk.urdf (robot description, URDF)
Before this commit: robot SM_Cup_object, 1 links, 0 joints
Links:
- removed link SM_Cup_main
- added link milk_main, mass 0.1; collision mesh filename=/home/user/catkin_init_ws/src/pycram/resources/milk.stl scale=1 1 1; visual mesh filename=/home/user/catkin_init_ws/src/pycram/resources/milk.stl scale=1 1 1
